File: proj1-rf24breakout/rf24-breakout-v1.kicad_pcb (KiCad board)
At the start: 2 copper layers, 33 x 17.8 mm, 2 parts, among them U1 nRF24

Commit message: First project complete with notes.
Parts:
- removed ?: CONN_01X08, Pin_Headers:Pin_Header_Straight_1x08
- added C1: 1uF, Capacitors_SMD:c_elec_8x10.5, F.Cu at (178.1, 97.0)
- added P1: CONN_01X08, Pin_Headers:Pin_Header_Straight_1x08, F.Cu at (170.8, 99.1)
Connections:
- U1 pad 0: /GND -> GND
Routing:
- net GND: track 0.00 -> 41.3 mm
- net /GND: track 23.4 -> 0.00 mm
- net /Vcc: track 33.1 -> 56.3 mm
- added copper zone on F.Cu, net GND
Other:
- board size 33 x 17.8 mm -> 33 x 21.8 mm
- net class Default: clearance 0.2 -> 0.1524; trace_width 0.25 -> 0.1524; via_dia 0.6 -> 0.6858; via_drill 0.4 -> 0.3302
- rule trace_clearance: 0.2 -> 0.1524
- rule trace_min: 0.2 -> 0.1524
- rule via_min_drill: 0.3 -> 0.3302
- rule via_min_size: 0.4 -> 0.6858
- board text added: "CE"
- board text added: "CSN"
- board text added: "GND"
- board text added: "IRQ"
- board text added: "MISO"
- board text added: "MOSI"
- board text added: "SCK"
- board text added: "Vcc"
- board text added: "v1.1"
